File: kicad/_autosave-funkydude-smd.kicad_pcb (KiCad board)
At the start: 2 copper layers, 40.6 x 29 mm, 33 parts, among them P1 CONN_2, P2 CONN_2, P3 CONN_2, SW1 SWITCH_INV, SW2 SWITCH_INV, U1 OP284

Commit message: Signed-off-by: Dolganoff <adolganov@gmail.com>
Other:
- net class Default: via_dia 0.889 -> 0.762; via_drill 0.635 -> 0.508
- rule via_min_size: 0.889 -> 0.762
- board text added: "V1"
