File: kicad/funkydude-smd.kicad_pcb (KiCad board)
At the start: 2 copper layers, 40.6 x 29 mm, 33 parts, among them P1 CONN_2, P2 CONN_2, P3 CONN_2, SW1 SWITCH_INV, SW2 SWITCH_INV, U1 OP284

Commit message: Signed-off-by: Dolganoff <adolganov@gmail.com>
Other:
- board text added: "V1"

Commit message: Signed-off-by: Dolganoff <adolganov@gmail.com>
Other:
- net class Default: via_dia 0.889 -> 0.762; via_drill 0.635 -> 0.508
- rule via_min_size: 0.889 -> 0.762
Changed lines of the file:
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@@
     (links 56)
     (no_connects 0)
-    (area 97.211848 82.728999 141.299001 111.835001)
+    (area 100.508999 82.728999 141.299001 111.835001)
     (thickness 1.6)
     (drawings 9)
@@
     (35 F.Paste user)
     (36 B.SilkS user)
-    (37 F.SilkS user hide)
+    (37 F.SilkS user)
     (38 B.Mask user)
     (39 F.Mask user)
@@
     (segment_width 0.2)
     (edge_width 0.15)
-    (via_size 0.889)
-    (via_drill 0.635)
-    (via_min_size 0.889)
+    (via_size 0.762)
+    (via_drill 0.508)
+    (via_min_size 0.762)
     (via_min_drill 0.508)
     (uvia_size 0.508)
@@
     (clearance 0.254)
     (trace_width 0.381)
-    (via_dia 0.889)
-    (via_drill 0.635)
+    (via_dia 0.762)
+    (via_drill 0.508)
     (uvia_dia 0.508)
     (uvia_drill 0.127)
