File: src/kicad-tth/funky dude.sch (KiCad schematic (older format))
At the start: 33 parts, among them P1 CONN_2, P2 CONN_2, P3 CONN_2, SW1 SWITCH_INV, SW2 SWITCH_INV, U1 OP284

Commit message: version_2.0 initial
Connections:
- wire segments 101 -> 77
Changed lines of the file:
@@
 	2050 4050 2500 4050
 Wire Wire Line
-	6400 3400 6450 3400
-Wire Wire Line
-	6450 3400 6800 3400
-Wire Wire Line
-	6800 3400 7100 3400
+	6400 3400 7100 3400
 Wire Wire Line
 	8500 4900 8500 4600
 Wire Wire Line
-	8200 4600 8500 4600
-Wire Wire Line
-	8500 4600 8800 4600
-Wire Wire Line
-	8800 4600 8950 4600
-Wire Wire Line
-	9500 1900 9500 2450
-Wire Wire Line
-	9500 2450 9500 2600
+	8200 4600 8950 4600
+Wire Wire Line
+	9500 1900 9500 2600
 Connection ~ 6800 1900
 Wire Wire Line
@@
 Connection ~ 6450 3400
 Wire Wire Line
-	6450 2450 6450 2600
-Wire Wire Line
-	6450 2600 6450 3400
+	6450 2450 6450 3400
 Wire Wire Line
 	4600 4250 4700 4250
@@
 	5700 2600 5250 2600
 Wire Wire Line
-	5250 2450 5250 2600
-Wire Wire Line
-	5250 2600 5250 3500
-Wire Wire Line
-	5200 3500 5250 3500
-Wire Wire Line
-	5250 3500 5400 3500
+	5250 2450 5250 3500
+Wire Wire Line
+	5200 3500 5400 3500
 Connection ~ 5250 3500
 Wire Wire Line
@@
 Connection ~ 6450 1900
 Wire Wire Line
-	4550 3500 4600 3500
-Wire Wire Line
-	4600 3500 4700 3500
+	4550 3500 4700 3500
 Connection ~ 4600 3500
 Wire Wire Line
 	7000 4450 7000 4550
 Wire Wire Line
-	7000 3500 7000 3950
-Wire Wire Line
-	7000 3950 7000 4050
-Wire Wire Line
-	7000 4550 2750 4550
-Wire Wire Line
-	2750 4550 2750 3400
+	7000 3500 7000 4050
+Wire Wire Line
+	7000 4550 2700 4550
+Wire Wire Line
+	2700 4550 2700 3400
 Wire Wire Line
 	7600 2650 7500 2650
@@
 	7750 2200 7900 2200
 Wire Wire Line
-	7900 5000 7900 5100
-Wire Wire Line
-	7900 5100 7900 5150
+	7900 5000 7900 5150
 Wire Wire Line
 	7900 5100 8200 5100
@@
 	8500 5600 8500 5300
 Wire Wire Line
-	7900 5600 8200 5600
-Wire Wire Line
-	8200 5600 8500 5600
-Wire Wire Line
-	8500 5600 8800 5600
-Wire Wire Line
-	8800 5600 8950 5600
+	7900 5600 8950 5600
 Wire Wire Line
 	7900 5600 7900 5550
@@
 Connection ~ 8200 5100
 Wire Wire Line
-	7550 3450 7750 3450
-Wire Wire Line
-	7750 3450 7950 3450
+	7550 3450 7950 3450
 Wire Wire Line
 	2500 4050 2500 4250
@@
 $EndComp
 Wire Wire Line
-	3150 3400 3200 3400
-Wire Wire Line
-	3200 3400 3550 3400
+	3150 3400 3550 3400
 $Comp
 L GND #PWR010
@@
 	3400 3600 3550 3600
 Wire Wire Line
-	3400 2700 3400 2750
-Wire Wire Line
-	3400 2750 3400 3650
+	3400 2700 3400 3650
 Wire Wire Line
 	3200 3900 3200 4200
 Wire Wire Line
-	3200 4200 3400 4200
-Wire Wire Line
-	3400 4200 3500 4200
+	3200 4200 3500 4200
 Wire Wire Line
 	3400 4200 3400 4150
@@
 	4600 2750 4250 2750
 Wire Wire Line
-	3750 2200 3600 2200
-Wire Wire Line
-	3600 2200 3400 2200
+	3400 2200 3750 2200
 Wire Wire Line
 	4250 2200 4600 2200
@@
 Connection ~ 9500 2450
 Wire Wire Line
-	5250 1900 6450 1900
-Wire Wire Line
-	6450 1900 6800 1900
-Wire Wire Line
-	6800 1900 8450 1900
-Wire Wire Line
-	8450 1900 8550 1900
+	5250 1900 8550 1900
 Wire Wire Line
 	8450 2150 8350 2150
@@
 $EndComp
 Wire Wire Line
-	4600 2200 4600 2750
-Wire Wire Line
-	4600 2750 4600 3500
-Wire Wire Line
-	4600 3500 4600 3550
+	4600 2200 4600 3550
 Wire Wire Line
 	4600 4050 4600 4250
@@
 	8350 3650 8400 3650
 Connection ~ 3400 3600
+Connection ~ 2700 3400
 $EndSCHEMATC

Commit message: 2014-10-22
Parts:
- removed C11: 47nf, User:C2-LARGE_PADS, symbol C
- removed SW1, SW2: SWITCH_INV, User:SIL-3-LARGE_PADS, symbol SWITCH_INV
- C1, C13, C2, C3, C4, C5, C6: footprint User:C2-LARGE_PADS -> Custom:C2-LARGE_PADS
- C10, C12, C8, C9: footprint User:C1V7-LARGE_PADS -> Custom:C1V5-LARGE_PADS
- C7: value 47uf -> 1uF; footprint User:C1V7-LARGE_PADS -> Custom:C1V5-LARGE_PADS
- P1, P2, P3: footprint User:SIL-2-LARGE_PADS -> Custom:SIL-2-LARGE_PADS
- R1, R10, R11, R2, R3, R5, R6, R7, R9: footprint User:R3-LARGE_PADS -> Custom:R3-LARGE_PADS
- R4: footprint User:R4-LARGE_PADS -> Custom:R3-LARGE_PADS
- R8: value 1Meg -> 470; footprint User:R3-LARGE_PADS -> Custom:R3-LARGE_PADS
- RBASS1, RTREBLE1: footprint User:SIL-3-LARGE_PADS -> Custom:SIL-3-LARGE_PADS
- U1: footprint User:DIP-8_LARGE_PADS -> Custom:DIP-8_LARGE_PADS
Connections:
- wire segments 77 -> 65
Other:
- moved on the sheet: C1, C10, C12, C13, C2, C3, C4, C5, C6, C8, C9, P1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
